File: rp2040/cpu.kicad_sch (KiCad schematic)
At the start: 27 parts, among them J3 Conn_02x05_SWD, SW9 Switch_SW_Push, U1 RP2040, U11 W25Q128JVS, X1 12MHz

Commit message: rp2040: update to kicad 9.0.2
Parts:
- C1, C2: value 20pF,50V,C0G -> 20pF,50V,C0G
- C10, C11, C12, C13, C14, C3, C4, C6, C7, C8: value 100nF,16V,X7R -> 100nF,16V,X7R
- C23: value 2.2uF,6.3V,X5R -> 2.2uF,6.3V,X5R
- C5: value 10uF,6.3V,X5R -> 10uF,6.3V,X5R
